Commit message: feat: added finger qpoints

File: f3rm_robot/assets/hithand_palm/hithand.urdf (robot description, URDF)
Before this commit: robot hithand, 23 links, 22 joints
Links:
- added link f3rm_grasp
- added link f3rm_index
- added link f3rm_little
- added link f3rm_middle
- added link f3rm_ring
- added link f3rm_thumb
Joints:
- added joint hithand_f3rm_grasp: type fixed, parent base_link_hithand, child f3rm_grasp, origin xyz=0.045 0 0.15 rpy=3.1416 0 1.5708
- added joint hithand_f3rm_index: type fixed, parent Right_Index_Phamed, child f3rm_index, origin xyz=0 0.02 0 rpy=0 0 0
- added joint hithand_f3rm_little: type fixed, parent Right_Little_Phamed, child f3rm_little, origin xyz=0 0.02 0 rpy=0 0 0
- added joint hithand_f3rm_middle: type fixed, parent Right_Middle_Phamed, child f3rm_middle, origin xyz=0 0.02 0 rpy=0 0 0
- added joint hithand_f3rm_ring: type fixed, parent Right_Ring_Phamed, child f3rm_ring, origin xyz=0 0.02 0 rpy=0 0 0
- added joint hithand_f3rm_thumb: type fixed, parent Right_Thumb_Phamed, child f3rm_thumb, origin xyz=0 0.02 0 rpy=0 0 0

Commit message: feat: added qp to all finger links, sh script to generate tasks

File: f3rm_robot/assets/hithand_palm/hithand.urdf (robot description, URDF)
Before this commit: robot hithand, 29 links, 28 joints
Links:
- removed link f3rm_index
- removed link f3rm_little
- removed link f3rm_middle
- removed link f3rm_ring
- removed link f3rm_thumb
- added link f3rm_index_dist
- added link f3rm_index_med
- added link f3rm_index_prox
- added link f3rm_little_dist
- added link f3rm_little_med
- added link f3rm_little_prox
- added link f3rm_middle_dist
- added link f3rm_middle_med
- added link f3rm_middle_prox
- added link f3rm_ring_dist
- added link f3rm_ring_med
- added link f3rm_ring_prox
- added link f3rm_thumb_dist
- added link f3rm_thumb_med
- added link f3rm_thumb_prox
Joints:
- removed joint hithand_f3rm_index
- removed joint hithand_f3rm_little
- removed joint hithand_f3rm_middle
- removed joint hithand_f3rm_ring
- removed joint hithand_f3rm_thumb
- added joint hithand_f3rm_index_dist: type fixed, parent Right_Index_Phadist, child f3rm_index_dist, origin xyz=-0.015 0.0175 0 rpy=0 0 0
- added joint hithand_f3rm_index_med: type fixed, parent Right_Index_Phamed, child f3rm_index_med, origin xyz=0 0.015 0 rpy=0 0 0
- added joint hithand_f3rm_index_prox: type fixed, parent Right_Index_Phaprox, child f3rm_index_prox, origin xyz=0.03 0.0175 0 rpy=0 0 0
- added joint hithand_f3rm_little_dist: type fixed, parent Right_Little_Phadist, child f3rm_little_dist, origin xyz=-0.015 0.0175 0 rpy=0 0 0
- added joint hithand_f3rm_little_med: type fixed, parent Right_Little_Phamed, child f3rm_little_med, origin xyz=0 0.015 0 rpy=0 0 0
- added joint hithand_f3rm_little_prox: type fixed, parent Right_Little_Phaprox, child f3rm_little_prox, origin xyz=0.03 0.0175 0 rpy=0 0 0
- added joint hithand_f3rm_middle_dist: type fixed, parent Right_Middle_Phadist, child f3rm_middle_dist, origin xyz=-0.015 0.0175 0 rpy=0 0 0
- added joint hithand_f3rm_middle_med: type fixed, parent Right_Middle_Phamed, child f3rm_middle_med, origin xyz=0 0.015 0 rpy=0 0 0
- added joint hithand_f3rm_middle_prox: type fixed, parent Right_Middle_Phaprox, child f3rm_middle_prox, origin xyz=0.03 0.0175 0 rpy=0 0 0
- added joint hithand_f3rm_ring_dist: type fixed, parent Right_Ring_Phadist, child f3rm_ring_dist, origin xyz=-0.015 0.0175 0 rpy=0 0 0
- added joint hithand_f3rm_ring_med: type fixed, parent Right_Ring_Phamed, child f3rm_ring_med, origin xyz=0 0.015 0 rpy=0 0 0
- added joint hithand_f3rm_ring_prox: type fixed, parent Right_Ring_Phaprox, child f3rm_ring_prox, origin xyz=0.03 0.0175 0 rpy=0 0 0
- added joint hithand_f3rm_thumb_dist: type fixed, parent Right_Thumb_Phadist, child f3rm_thumb_dist, origin xyz=-0.015 0.0175 0 rpy=0 0 0
- added joint hithand_f3rm_thumb_med: type fixed, parent Right_Thumb_Phamed, child f3rm_thumb_med, origin xyz=0 0.015 0 rpy=0 0 0
- added joint hithand_f3rm_thumb_prox: type fixed, parent Right_Thumb_Phaprox, child f3rm_thumb_prox, origin xyz=0.03 0.0175 0 rpy=0 0 0
